File: Motherboard/Hardware/Silverworm - CM5 Motherboard/CM5IO.kicad_pcb (KiCad board)
At the start: 4 copper layers, 160 x 90 mm, 79 parts, among them J10 690-019-298-412, J11 USB_C_Receptacle_USB2.0, J12 USB3_A, J14 JST_SHBM04B-SRSS-TB, J16 Conn_01x22_Female, J2 Conn_02x07_Odd_Even, J22 690-019-298-412, J3 Conn_01x03, J4 Bus_M.2_Socket_M, J5 Conn_01x22_Female, J6 THD-02-R, J7 Micro_SD_Card_Det, J8 THD-20-R, J9 THD-02-R, SW1 Right angle Tact button, U1 TPD4EUSB30, U12 RT9742SNGV, U18 RT9742GGJ5, U2 TPD4EUSB30, U3 MagJack-A70-112-331N126, U6 AP22653W6, U7 ASEK-32.768KHZ-L-R-T, U8 AP3441SHE-7B

Commit message: Motherboard schematics edits
Parts:
- removed BT1: Battery_Cell, CM5IO:BatteryHolder_Keystone_3034_1x20mm
- added R18: 5.1K, Resistor_SMD:R_0402_1005Metric, F.Cu at (160.1, 173.7)
- added R19: 5.1K, Resistor_SMD:R_0402_1005Metric, F.Cu at (160.1, 175.7)
- added R20: 649R, Resistor_SMD:R_0402_1005Metric, F.Cu at (165.0, 173.7)
Connections:
- C12 pad 1: /+5v -> /CM5_HighSpeed/+5v
- C2 pad 1: /+5v -> /CM5_HighSpeed/+5v
- J11 pad A6: /USB2_P -> Net-(J11-D+-PadA6)
- J11 pad A7: /USB2_N -> Net-(J11-D--PadA7)
- J11 pad B6: /USB2_P -> Net-(J11-D+-PadA6)
- J11 pad B7: /USB2_N -> Net-(J11-D--PadA7)
- J16 pad 22: /+3.3v -> /CM5_HighSpeed/+3.3v
- J5 pad 22: /+3.3v -> /CM5_HighSpeed/+3.3v
- Module1 pad 103: /USB2_N -> /CM5_HighSpeed/USB2_N
- Module1 pad 105: /USB2_P -> /CM5_HighSpeed/USB2_P
- R8 pad 1: /+3.3v -> /CM5_HighSpeed/+3.3v
- R9 pad 1: /+5v -> GND
- R9 pad 2: GND -> /+5v
- U12 pad 1: /+5v -> /CM5_HighSpeed/+5v
- U6 pad 1: /+5v -> /CM5_HighSpeed/+5v
Routing:
- net (no net): track 0.00 -> 143.6 mm, vias 0 -> 4
- net /USB2_N: track 71.9 -> 0.00 mm, vias 2 -> 0
- net /USB2_P: track 71.7 -> 0.00 mm, vias 2 -> 0
Other:
- board text removed: "Battery CR2032"
