File: Motherboard/Hardware/Silverworm - CM5 Motherboard/CM5IO.kicad_pcb (KiCad board)
At the start: 4 copper layers, 89 parts, among them J1 USB_C_Receptacle_USB2.0, J10 Conn_01x03, J11 THD-20-R, J12 Microfit 3-pin, J13 THD-02-R, J14 Microfit 6-pin, J15 Microfit 2-Pin, J16 Microfit 2-Pin, J17 Microfit 2-Pin, J18 Microfit 2-Pin, J2 Conn_01x22_Female, J20 USB_A, J23 Mega-Fit-1row-2pin, J24 Mega-Fit-2row-2pin, J3 Conn_01x22_Female, J4 THD-02-R, J5 USB3_A, J6 690-019-298-412, J7 690-019-298-412, J8 Conn_02x07_Odd_Even, J9 JST_SHBM04B-SRSS-TB, SW1 Right angle Tact button, U1 AP22653W6, U10 10uH, U2 RT9742SNGV, U3 TPD4EUSB30, U4 TPD4EUSB30, U5 MagJack-A70-112-331N126, U9 SS54

Commit message: motherboard layout
Parts:
- removed H8: MountingHole, CM5IO:MountingHole_2.7mm_M2.5_DIN965
- removed TP1: TestPoint, TestPoint:TestPoint_Pad_2.0x2.0mm
- added C18: 100n, Capacitor_SMD:C_0402_1005Metric, F.Cu at (193.7, 150.8)
- added C19: GVT1J476M0608CNVC, Capacitor_SMD:CP_Elec_6.3x7.7, F.Cu at (219.5, 100.2)
- added TP5: TestPoint, TestPoint:TestPoint_Pad_2.0x2.0mm, B.Cu at (116.6, 155.8)
- added U8: TPS54560DDAR, TPS54560DDAR:SOIC127P600X170-9N, F.Cu at (229.5, 93.7)
- J15, J16, J17, J18: footprint Connector_Molex:Molex_Micro-Fit_3.0_43650-0215_1x02_P3.00mm_Vertical -> Connector_Molex:Molex_Micro-Fit_3.0_43045-0221_2x01-1MP_P3.00mm_Horizontal
- TP2, TP3, TP4: moved to B.Cu
- moved C7 308.6 mm to (357.0, 107.2)
- moved C8 308.6 mm to (357.0, 109.2)
- moved R9 294.0 mm to (361.8, 86.2)
- moved C5 283.3 mm to (361.8, 79.2)
- moved C6 283.3 mm to (361.8, 82.2)
- moved R4 279.7 mm to (354.1, 107.2)
- moved R5 279.7 mm to (354.1, 109.2)
- moved R8 276.6 mm to (344.5, 107.2)
- moved R13 276.5 mm to (344.5, 109.2)
- moved SPI_1 230.1 mm to (260.2, 95.8), turned to -90 degrees
- moved J18 224.0 mm to (254.2, 151.9), turned to 180 degrees
- moved C23 214.9 mm to (326.6, 82.5)
- moved C25 214.9 mm to (326.6, 85.9)
- moved C26 214.9 mm to (326.6, 89.2)
- moved D4 214.9 mm to (326.7, 92.6)
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Routing:
- net 24V_INPUT: track 184.7 -> 0.00 mm, vias 4 -> 0
- net GND: track 866.1 -> 694.0 mm, vias 455 -> 431
- net /CM5_GPIO ( Ethernet, GPIO, SDCARD)/VBAT: track 154.9 -> 0.00 mm, vias 2 -> 0
- net (no net): track 231.7 -> 87.2 mm, vias 13 -> 3
- net +24V: track 138.2 -> 0.00 mm, vias 4 -> 0
- net /CM5_HighSpeed/USB2_N: track 194.2 -> 71.9 mm, vias 3 -> 2
- net /CM5_GPIO ( Ethernet, GPIO, SDCARD)/GPIO2: track 0.00 -> 122.2 mm, vias 0 -> 1
- net +5V: track 341.9 -> 224.7 mm, vias 29 -> 19
- net /CM5_GPIO ( Ethernet, GPIO, SDCARD)/LED_DATA: track 0.00 -> 117.2 mm, vias 0 -> 1
- net /CM5_GPIO ( Ethernet, GPIO, SDCARD)/GPIO14: track 117.2 -> 0.00 mm, vias 1 -> 0
- net /CM5_GPIO ( Ethernet, GPIO, SDCARD)/GPIO4: track 116.1 -> 0.00 mm, vias 1 -> 0
- net /CM5_GPIO ( Ethernet, GPIO, SDCARD)/CSn_3: track 0.00 -> 116.1 mm, vias 0 -> 1
- net /CM5_GPIO ( Ethernet, GPIO, SDCARD)/CSn_1: track 0.00 -> 113.6 mm, vias 0 -> 1
- net /CM5_GPIO ( Ethernet, GPIO, SDCARD)/GPIO18: track 113.6 -> 0.00 mm, vias 1 -> 0
- net /CM5_GPIO ( Ethernet, GPIO, SDCARD)/LK_4: track 0.00 -> 110.5 mm
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- added copper zone on B.Cu, net (none)
- added copper zone on F.Cu, net (none)
- added copper zone on B.Cu, net /CM5_HighSpeed/HDMI_5v
- added copper zone on F.Cu, net /CM5_HighSpeed/SCL1
- removed copper zone on B.Cu, net +5V
- removed copper zone on F.Cu, net +5V
- removed copper zone on B.Cu, net VBUS
Other:
- board outline added: 190 x 90 mm
- board text added: "CAM/DISP 0"
- board text added: "CAM/DISP 1"
- board text added: "Compute Module 5"
- board text added: "Compute Module 5 IO Board"
- board text added: "Ethernet"
- board text added: "FAN"
- board text added: "Fit for 1.8V GPIO"
- board text added: "Fit for 3.3V GPIO"
- board text added: "Fit jumper to disable eMMC Boot"
- board text added: "Fit jumper to disable writing to EEPROM"
- board text added: "Fit two jumpers for CAM/DISP 1"
- board text added: "HDMI0"
- board text added: "HDMI1"
- board text added: "J3 : nBT_Dis GND"
- board text added: "PMIC_Enable"
- board text added: "POE"
- board text added: "PWR_Button"
- board text added: "Power Button"
- board text added: "Power In"
- board text added: "Raspberry Pi HAT"
- board text added: "SYNC_Out"
- board text added: "USB Device"
- board text added: "USB3"
- board text added: "USB_OTG"
- board text added: "nWireless_Dis"
- board text removed: "Designed by Zak Leek © 2026"
- board text removed: "Silverworm Motherboard For RPi CM5"
- board text removed: "Why are you loking at my bottom? ;)"
