File: Motherboard/Hardware/Silverworm - CM5 Motherboard/CM5_HighSpeed.kicad_sch (KiCad schematic)
At the start: 19 parts, among them J10 690-019-298-412, J12 USB3_A, J16 Conn_01x22_Female, J22 690-019-298-412, J5 Conn_01x22_Female, J6 THD-02-R, U12 RT9742SNGV, U6 AP22653W6

Commit message: Motherboard schematics edits
Connections:
- net PCIE_CLK_N: no longer names the net of Module1.112 (PCIe_CLK_N)
- net PCIE_CLK_P: no longer names the net of Module1.110 (PCIe_CLK_P)
- net PCIE_PWR_EN: no longer names the net of Module1.106 (PCIE_PWR_EN)
- net PCIE_RX_N: no longer names the net of Module1.118 (PCIe_RX_N)
- net PCIE_RX_P: no longer names the net of Module1.116 (PCIe_RX_P)
- net PCIE_TX_N: no longer names the net of Module1.124 (PCIe_TX_N)
- net PCIE_TX_P: no longer names the net of Module1.122 (PCIe_TX_P)
- net PCIE_nCLKREQ: no longer names the net of Module1.102 (PCIe_nCLKREQ)
- net PCIE_nRST: no longer names the net of Module1.109 (PCIe_nRST)
- net PCIE_nWAKE: no longer names the net of Module1.104 (PCIE_nWAKE)
Other:
- company: Copyright © 2024 Raspberry Pi Ltd. -> Copyright © Zak Leek, Imperial College London
- title: Compute Module 5 IO Board - CM5 - Highspeed -> Compute Module 5 IO Board - Top Level
Changed lines of the file:
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@@
 	(paper "A4")
 	(title_block
-		(title "Compute Module 5 IO Board - CM5 - Highspeed")
+		(title "Compute Module 5 IO Board - Top Level")
+		(date "2026-01-27")
 		(rev "1")
-		(company "Copyright © 2024 Raspberry Pi Ltd.")
-		(comment 1 "www.raspberrypi.com")
+		(company "Copyright © Zak Leek, Imperial College London")
+		(comment 1 "DMT4 - Silerworm, Group 4C")
 	)
 	(text "USB 3 Pairs P/N swapped to help routing"
@@
 	(wire
 		(pts
-			(xy 31.75 38.1) (xy 38.1 38.1)
-		)
-		(stroke
-			(width 0)
-			(type solid)
-		)
-	)
-	(wire
-		(pts
 			(xy 35.56 109.22) (xy 38.1 109.22)
 		)
@@
 	(wire
 		(pts
-			(xy 31.75 27.94) (xy 38.1 27.94)
-		)
-		(stroke
-			(width 0)
-			(type default)
-		)
-	)
-	(wire
-		(pts
 			(xy 180.34 48.26) (xy 196.85 48.26)
 		)
@@
 	(wire
 		(pts
-			(xy 38.1 43.18) (xy 31.75 43.18)
-		)
-		(stroke
-			(width 0)
-			(type solid)
-		)
-	)
-	(wire
-		(pts
 			(xy 99.06 76.2) (xy 115.57 76.2)
 		)
@@
 	(wire
 		(pts
-			(xy 31.75 30.48) (xy 38.1 30.48)
-		)
-		(stroke
-			(width 0)
-			(type default)
-		)
-	)
-	(wire
-		(pts
 			(xy 99.06 132.08) (xy 101.6 132.08)
 		)
@@
 	(wire
 		(pts
-			(xy 31.75 53.34) (xy 38.1 53.34)
-		)
-		(stroke
-			(width 0)
-			(type solid)
-		)
-	)
-	(wire
-		(pts
 			(xy 148.59 119.38) (xy 148.59 127)
 		)
@@
 	(wire
 		(pts
-			(xy 38.1 45.72) (xy 31.75 45.72)
-		)
-		(stroke
-			(width 0)
-			(type solid)
-		)
-	)
-	(wire
-		(pts
 			(xy 101.6 93.98) (xy 101.6 101.6)
 		)
@@
 	(wire
 		(pts
-			(xy 31.75 35.56) (xy 38.1 35.56)
-		)
-		(stroke
-			(width 0)
-			(type solid)
-		)
-	)
-	(wire
-		(pts
 			(xy 101.6 139.7) (xy 101.6 147.32)
 		)
@@
 	(wire
 		(pts
-			(xy 31.75 25.4) (xy 38.1 25.4)
-		)
-		(stroke
-			(width 0)
-			(type solid)
-		)
-	)
-	(wire
-		(pts
 			(xy 180.34 80.01) (xy 196.85 80.01)
 		)
@@
 	(wire
 		(pts
-			(xy 31.75 50.8) (xy 38.1 50.8)
-		)
-		(stroke
-			(width 0)
-			(type solid)
-		)
-	)
-	(wire
-		(pts
 			(xy 134.62 121.92) (xy 151.13 121.92)
 		)
@@
 	(wire
 		(pts
-			(xy 99.06 35.56) (xy 105.41 35.56)
-		)
-		(stroke
-			(width 0)
-			(type solid)
-		)
-	)
-	(wire
-		(pts
 			(xy 99.06 121.92) (xy 115.57 121.92)
 		)
@@
 		)
 	)
-	(hierarchical_label "PCIE_PWR_EN"
-		(shape output)
-		(at 31.75 30.48 180)
-		(effects
-			(font
-				(size 1.27 1.27)
-			)
-			(justify right)
-		)
-	)
-	(hierarchical_label "PCIE_CLK_P"
-		(shape output)
-		(at 31.75 35.56 180)
-		(effects
-			(font
-				(size 1.27 1.27)
-			)
-			(justify right)
-		)
-	)
 	(hierarchical_label "CAM_GPIO0"
 		(shape input)
@@
 		)
 	)
-	(hierarchical_label "PCIE_RX_N"
-		(shape input)
-		(at 31.75 45.72 180)
-		(effects
-			(font
-				(size 1.27 1.27)
-			)
-			(justify right)
-		)
-	)
 	(hierarchical_label "+5v"
 		(shape input)
@@
 		)
 	)
-	(hierarchical_label "PCIE_nCLKREQ"
-		(shape input)
-		(at 31.75 25.4 180)
-		(effects
-			(font
-				(size 1.27 1.27)
-			)
-			(justify right)
-		)
-	)
 	(hierarchical_label "ID_SC"
 		(shape input)
@@
 		)
 	)
-	(hierarchical_label "PCIE_RX_P"
-		(shape input)
-		(at 31.75 43.18 180)
-		(effects
-			(font
-				(size 1.27 1.27)
-			)
-			(justify right)
-		)
-	)
 	(hierarchical_label "GPIO_VREF"
 		(shape input)
@@
 		)
 	)
-	(hierarchical_label "PCIE_TX_P"
-		(shape output)
-		(at 31.75 50.8 180)
-		(effects
-			(font
-				(size 1.27 1.27)
-			)
-			(justify right)
-		)
-	)
 	(hierarchical_label "ID_SD"
 		(shape input)
@@
 		)
 	)
-	(hierarchical_label "PCIE_nWAKE"
-		(shape input)
-		(at 31.75 27.94 180)
-		(effects
-			(font
-				(size 1.27 1.27)
-			)
-			(justify right)
-		)
-	)
-	(hierarchical_label "PCIE_CLK_N"
-		(shape output)
-		(at 31.75 38.1 180)
-		(effects
-			(font
-				(size 1.27 1.27)
-			)
-			(justify right)
-		)
-	)
-	(hierarchical_label "PCIE_nRST"
-		(shape output)
-		(at 105.41 35.56 0)
-		(effects
-			(font
-				(size 1.27 1.27)
-			)
-			(justify left)
-		)
-	)
 	(hierarchical_label "CAM_GPIO1"
 		(shape input)
@@
 		(effects
 			(font
-				(size 1.27 1.27)
-			)
-			(justify right)
-		)
-	)
-	(hierarchical_label "PCIE_TX_N"
-		(shape output)
-		(at 31.75 53.34 180)
-		(effects
-			(font
