File: Motherboard/Hardware/Silverworm - CM5 Motherboard/CM5_HighSpeed.kicad_sch (KiCad schematic)
At the start: 19 parts, among them J10 690-019-298-412, J12 USB3_A, J16 Conn_01x22_Female, J22 690-019-298-412, J5 Conn_01x22_Female, J6 THD-02-R, U12 RT9742SNGV, U6 AP22653W6

Commit message: Layout and IO edits
Other:
- title: Compute Module 5 IO Board - Top Level -> Silverwom CM5 Motherboard - HighSpeed
Changed lines of the file:
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@@
 	(paper "A4")
 	(title_block
-		(title "Compute Module 5 IO Board - Top Level")
+		(title "Silverwom CM5 Motherboard - HighSpeed")
 		(date "2026-01-27")
 		(rev "1")

Commit message: PCB changes (many)
Parts:
- renumbered C2 to C3, C3 to C4, C7 to C5, C8 to C6, C12 to C7, C13 to C8, J5 to J2, J16 to J3, J6 to J4, J12 to J5, J22 to J6, J10 to J7, R12 to R4, R8 to R5, U6 to U1, U12 to U2
Connections:
- net +5v renamed +5V
