File: Motherboard/Hardware/Silverworm - CM5 Motherboard/PCIe-M2.kicad_sch (KiCad schematic)
At the start: 24 parts, among them J4 Bus_M.2_Socket_M, M1 M.2 Screw, M2 M.2 Solder Nut, M3 M.2 Solder Nut, M4 M.2 Solder Nut, M5 M.2 Solder Nut, U7 ASEK-32.768KHZ-L-R-T, U8 AP3441SHE-7B

Commit message: Motherboard schematics edits
Other:
- company: Copyright © 2024 Raspberry Pi Ltd. -> Copyright © Zak Leek, Imperial College London
- title: Compute Module 5 IO Board - M2 Socket -> Compute Module 5 IO Board - Top Level
Changed lines of the file:
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@@
 	(paper "A4")
 	(title_block
-		(title "Compute Module 5 IO Board - M2 Socket")
+		(title "Compute Module 5 IO Board - Top Level")
+		(date "2026-01-27")
 		(rev "1")
-		(company "Copyright © 2024 Raspberry Pi Ltd.")
-		(comment 1 "www.raspberrypi.com")
+		(company "Copyright © Zak Leek, Imperial College London")
+		(comment 1 "DMT4 - Silerworm, Group 4C")
 	)
 	(text "Activity LED"
