File: Motherboard/Hardware/Silverworm - CM5 Motherboard/CM5IO_archive.kicad_pcb (KiCad board)
At the start: 4 copper layers, 89 parts, among them J1 USB_C_Receptacle_USB2.0, J10 Conn_01x03, J11 THD-20-R, J12 Microfit 3-pin, J13 THD-02-R, J14 Microfit 6-pin, J15 Microfit 2-Pin, J16 Microfit 2-Pin, J17 Microfit 2-Pin, J18 Microfit 2-Pin, J2 Conn_01x22_Female, J20 USB_A, J23 Mega-Fit-1row-2pin, J24 Mega-Fit-2row-2pin, J3 Conn_01x22_Female, J4 THD-02-R, J5 USB3_A, J6 690-019-298-412, J7 690-019-298-412, J8 Conn_02x07_Odd_Even, J9 JST_SHBM04B-SRSS-TB, SW1 Right angle Tact button, U1 AP22653W6, U10 10uH, U2 RT9742SNGV, U3 TPD4EUSB30, U4 TPD4EUSB30, U5 MagJack-A70-112-331N126, U9 SS54

Commit message: PCB changes (many)
Parts:
- added C10: 100n, Capacitor_SMD:C_0402_1005Metric, F.Cu at (224.1, 130.5)
- added C11: 4.7nF, Capacitor_SMD:C_0402_1005Metric, F.Cu at (222.4, 129.3)
- added C12: 100n, Capacitor_SMD:C_0402_1005Metric, F.Cu at (111.5, 149.5)
- added C13: 100n, Capacitor_SMD:C_0402_1005Metric, F.Cu at (116.8, 148.6)
- added C14: 10u, Capacitor_SMD:C_0805_2012Metric, F.Cu at (230.2, 126.4)
- added C15: 10u, Capacitor_SMD:C_0805_2012Metric, F.Cu at (230.2, 132.4)
- added C16: 10u, Capacitor_SMD:C_0805_2012Metric, F.Cu at (230.2, 130.4)
- added C17: 10u, Capacitor_SMD:C_0805_2012Metric, F.Cu at (230.1, 128.4)
- added C18: 100n, Capacitor_SMD:C_0402_1005Metric, F.Cu at (242.4, 149.3)
- added C19: GVT1J476M0608CNVC, Capacitor_SMD:C_0402_1005Metric, F.Cu at (226.7, 135.7)
- added D3: LED Green, LED_SMD:LED_0603_1608Metric, F.Cu at (229.1, 149.3)
- added IC1: CY7C65632-28LTXC, CM5IO:QFN50P500X500X80-29N-D, F.Cu at (203.5, 136.7)
- added J22: 690-019-298-412, CM5IO:EDAC 690-019-298-412, F.Cu at (102.0, 150.4)
- added L1: 2.2uH, CM5IO:L_Bourns_SRP5030CC, F.Cu at (228.7, 121.1)
- added R20: 649R, Resistor_SMD:R_0402_1005Metric, F.Cu at (197.0, 139.2)
- added SPI_3: Minifit 2x4, Connector_Molex:Molex_Mini-Fit_Jr_5569-08A2_2x04_P4.20mm_Horizontal, F.Cu at (249.2, 97.0)
- added TP5: TestPoint, TestPoint:TestPoint_Pad_2.0x2.0mm, B.Cu at (113.1, 156.1)
- added U12: RT9742SNGV, Package_TO_SOT_SMD:TSOT-23_HandSoldering, F.Cu at (114.1, 147.6)
- added U18: RT9742GGJ5, Package_TO_SOT_SMD:SOT-23-5, F.Cu at (206.9, 93.3)
- added U6: AP22653W6, Package_TO_SOT_SMD:SOT-23-6, F.Cu at (206.4, 102.3)
- added U7: ASEK-32.768KHZ-L-R-T, Crystal:Crystal_SMD_3225-4Pin_3.2x2.5mm, F.Cu at (229.2, 136.6)
- added U8: TPS54560DDAR, Package_DFN_QFN:DFN-8-1EP_2x2mm_P0.5mm_EP1.05x1.75mm, F.Cu at (226.2, 127.4)
- J16: footprint Connector_Molex:Molex_Micro-Fit_3.0_43650-0215_1x02_P3.00mm_Vertical -> CM5IO:Hirose_FH12-22S-0.5SH_1x22-1MP_P0.50mm_Horizontal
- J5: footprint CM5IO:MTCONN_UBAF30-D2011 -> CM5IO:Hirose_FH12-22S-0.5SH_1x22-1MP_P0.50mm_Horizontal
- J9: footprint Connector_JST:JST_SH_BM04B-SRSS-TB_1x04-1MP_P1.00mm_Vertical -> Connector_PinHeader_2.54mm:PinHeader_2x02_P2.54mm_Vertical
- TP1, TP2, TP3, TP4: moved to B.Cu
- U3: footprint Package_SON:USON-10_2.5x1.0mm_P0.5mm -> CM5IO:TRJG0926HENL
- moved J11 227.1 mm to (238.2, 155.7)
- moved SPI_1 220.3 mm to (249.2, 76.9), turned to -90 degrees
- moved J7 210.8 mm to (253.9, 138.2), turned to -90 degrees
- moved C4 208.8 mm to (226.7, 130.4)
- moved H1 197.2 mm to (277.5, 153.7)
- moved H4 191.6 mm to (278.0, 160.7)
- moved H3 190.8 mm to (278.5, 145.2)
- moved H2 188.8 mm to (271.5, 136.7), turned to 90 degrees
- moved H5 183.9 mm to (278.5, 138.7)
- moved H6 177.7 mm to (271.5, 152.2), turned to 90 degrees
- moved H8 172.7 mm to (271.5, 159.7), turned to 90 degrees
- moved Module1 172.1 mm to (195.5, 73.5), turned to 180 degrees
- moved H7 171.3 mm to (271.5, 144.2), turned to 90 degrees
- moved J4 168.8 mm to (147.8, 200.5)
- moved C9 168.0 mm to (236.4, 149.3), turned to 180 degrees
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Routing:
- net 24V_INPUT: track 184.7 -> 0.00 mm, vias 4 -> 0
- net (no net): track 231.7 -> 62.3 mm, vias 13 -> 0
- net +24V: track 138.2 -> 0.00 mm, vias 4 -> 0
- net /CM5_GPIO ( Ethernet, GPIO, SDCARD)/GPIO2: track 0.00 -> 122.2 mm, vias 0 -> 1
- net /CM5_HighSpeed/USB2_N: track 194.2 -> 71.9 mm, vias 3 -> 2
- net /PCIe-M2/M2_3v3: track 0.00 -> 99.8 mm, vias 0 -> 2
- net /CM5_HighSpeed/DPHY0_D1_N: track 0.00 -> 94.6 mm, vias 0 -> 2
- net /CM5_HighSpeed/DPHY0_C_N: track 0.00 -> 92.4 mm, vias 0 -> 2
- net /CM5_HighSpeed/DPHY0_C_P: track 0.00 -> 92.2 mm, vias 0 -> 2
- net /CM5_HighSpeed/DPHY0_D1_P: track 177.7 -> 94.5 mm, vias 3 -> 2
- net Net-(U5-LEDG_K): track 69.0 -> 0.00 mm
- net /CM5_GPIO ( Ethernet, GPIO, SDCARD)/SD_PWR: track 0.00 -> 68.1 mm
- net +12V: track 0.00 -> 43.5 mm
- net /+5v: track 0.00 -> 22.9 mm
- net Net-(IC1-DD-[3]): track 0.00 -> 22.5 mm, vias 0 -> 2
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Other:
- board outline added: 183 x 90 mm
- board text added: "CAM/DISP 0"
- board text added: "CAM/DISP 1"
- board text added: "Compute Module 5"
- board text added: "Ethernet"
- board text added: "FAN"
- board text added: "Fit for 1.8V GPIO"
- board text added: "Fit for 3.3V GPIO"
- board text added: "Fit jumper to disable eMMC Boot"
- board text added: "Fit jumper to disable writing to EEPROM"
- board text added: "Fit two jumpers for CAM/DISP 1"
- board text added: "HDMI0"
- board text added: "HDMI1"
- board text added: "J16"
- board text added: "J3 : nBT_Dis GND"
- board text added: "J5"
- board text added: "PMIC_Enable"
- board text added: "POE"
- board text added: "PWR_Button"
- board text added: "Power Button"
- board text added: "Power In"
- board text added: "R2"
- board text added: "Raspberry Pi HAT"
- board text added: "SYNC_Out"
- board text added: "USB Device"
- board text added: "USB3"
- board text added: "USB_OTG"
- board text added: "nWireless_Dis"
