File: Motherboard/Hardware/Silverworm - CM5 Motherboard/power_supply.kicad_sch (KiCad schematic)
At the start: 19 parts, among them J23 Mega-Fit-1row-2pin, J24 Mega-Fit-2row-2pin, U10 10uH, U8 TPS54560DDAR, U9 SS54

Commit message: motherboard layout
Parts:
- C19: footprint JLCPCB-Footprints:CAP-SMD_BD6.3-L6.6-W6.6-LS7.3-FD -> Capacitor_SMD:CP_Elec_6.3x7.7
- U8: footprint JLCPCB-Footprints:SOIC-8_L5.0-W4.0-P1.27-LS6.0-BL-EP2.0 -> TPS54560DDAR:SOIC127P600X170-9N
Changed lines of the file:
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@@
+		(dnp no)
+		(fields_autoplaced yes)
+		(property "Reference" "#PWR073"
+			(at 129.54 119.38 0)
+			(effects
+				(font
+					(size 1.27 1.27)
+				)
+				(hide yes)
+			)
+		)
+		(property "Value" "GND"
+			(at 129.54 118.11 0)
+			(effects
+				(font
+					(size 1.27 1.27)
+				)
+			)
+		)
+		(property "Footprint" ""
+			(at 129.54 113.03 0)
+			(effects
+				(font
+					(size 1.27 1.27)
+				)
+				(hide yes)
+			)
+		)
+		(property "Datasheet" ""
+			(at 129.54 113.03 0)
+			(effects
+				(font
+					(size 1.27 1.27)
+				)
+				(hide yes)
+			)
+		)
+		(property "Description" "Power symbol creates a global label with name \"GND\" , ground"
+			(at 129.54 113.03 0)
+			(effects
+				(font
+					(size 1.27 1.27)
+				)
+				(hide yes)
+			)
+		)
+		(pin "1"
+		)
+		(instances
+			(project ""
+				(path "/e63e39d7-6ac0-4ffd-8aa3-1841a4541b55/95be1478-6e3a-4dac-ad6d-2e684e4369ea"
+					(reference "#PWR073")
+					(unit 1)
+				)
+			)
+		)
+	)
+	(symbol
+		(lib_id "power:+5V")
+		(at 158.75 63.5 270)
+		(unit 1)
+		(exclude_from_sim no)
+		(in_bom yes)
+		(on_board yes)
 		(dnp no)
 		(fields_autoplaced yes)
 		(property "Reference" "#PWR074"
-			(at 129.54 119.38 0)
-			(effects
-				(font
-					(size 1.27 1.27)
-				)
-				(hide yes)
-			)
-		)
-		(property "Value" "GND"
-			(at 129.54 118.11 0)
-			(effects
-				(font
-					(size 1.27 1.27)
-				)
-			)
-		)
-		(property "Footprint" ""
-			(at 129.54 113.03 0)
-			(effects
-				(font
-					(size 1.27 1.27)
-				)
-				(hide yes)
-			)
-		)
-		(property "Datasheet" ""
-			(at 129.54 113.03 0)
-			(effects
-				(font
-					(size 1.27 1.27)
-				)
-				(hide yes)
-			)
-		)
-		(property "Description" "Power symbol creates a global label with name \"GND\" , ground"
-			(at 129.54 113.03 0)
-			(effects
-				(font
-					(size 1.27 1.27)
-				)
-				(hide yes)
-			)
-		)
-		(pin "1"
-		)
-		(instances
-			(project ""
-				(path "/e63e39d7-6ac0-4ffd-8aa3-1841a4541b55/95be1478-6e3a-4dac-ad6d-2e684e4369ea"
-					(reference "#PWR074")
-					(unit 1)
-				)
-			)
-		)
-	)
-	(symbol
-		(lib_id "power:+5V")
-		(at 158.75 63.5 270)
-		(unit 1)
-		(exclude_from_sim no)
-		(in_bom yes)
-		(on_board yes)
-		(dnp no)
-		(fields_autoplaced yes)
-		(property "Reference" "#PWR073"
 			(at 154.94 63.5 0)
 			(effects
@@
 			(project ""
 				(path "/e63e39d7-6ac0-4ffd-8aa3-1841a4541b55/95be1478-6e3a-4dac-ad6d-2e684e4369ea"
-					(reference "#PWR073")
+					(reference "#PWR074")
 					(unit 1)
 				)
@@
 			)
 		)
-		(property "Footprint" "JLCPCB-Footprints:CAP-SMD_BD6.3-L6.6-W6.6-LS7.3-FD"
+		(property "Footprint" "Capacitor_SMD:CP_Elec_6.3x7.7"
 			(at 33.02 71.12 0)
 			(effects
@@
 			)
 		)
-		(property "Footprint" "JLCPCB-Footprints:SOIC-8_L5.0-W4.0-P1.27-LS6.0-BL-EP2.0"
+		(property "Footprint" "TPS54560DDAR:SOIC127P600X170-9N"
 			(at 77.47 73.66 0)
 			(effects
