File: Motherboard/Hardware/Silverworm - CM5 Motherboard/Archived/CM5IO_dissassemled.kicad_pcb (KiCad board)
At the start: 4 copper layers, 183 x 90 mm, 111 parts, among them IC1 CY7C65632-28LTXC, J1 USB_C_Receptacle_USB2.0, J10 Conn_01x03, J11 THD-20-R, J12 Microfit 3-pin, J13 THD-02-R, J14 Microfit 6-pin, J15 Microfit 2-Pin, J16 Microfit 2-Pin, J17 Microfit 2-Pin, J18 Microfit 2-Pin, J2 Conn_01x22_Female, J20 USB_A, J22 690-019-298-412, J23 Mega-Fit-1row-2pin, J24 Mega-Fit-2row-2pin, J3 Conn_01x22_Female, J4 THD-02-R, J5 USB3_A, J6 690-019-298-412, J7 690-019-298-412, J8 Conn_02x07_Odd_Even, J9 JST_SHBM04B-SRSS-TB, SW1 Right angle Tact button, U1 AP22653W6, U10 10uH, U12 RT9742SNGV, U18 RT9742GGJ5, U2 RT9742SNGV, U3 TPD4EUSB30, U4 TPD4EUSB30, U5 MagJack-A70-112-331N126, U6 AP22653W6, U7 ASEK-32.768KHZ-L-R-T, U8 TPS54560DDAR, U9 SS54

Commit message: motherboard layout
Parts:
- removed C10, C12, C13, C18: 100n, Capacitor_SMD:C_0402_1005Metric
- removed C11: 4.7nF, Capacitor_SMD:C_0402_1005Metric
- removed C14, C15, C16, C17: 10u, Capacitor_SMD:C_0805_2012Metric
- removed C19: GVT1J476M0608CNVC, Capacitor_SMD:C_0402_1005Metric
- removed D3: LED Green, LED_SMD:LED_0603_1608Metric
- removed IC1: CY7C65632-28LTXC, CM5IO:QFN50P500X500X80-29N-D
- removed J22: 690-019-298-412, CM5IO:EDAC 690-019-298-412
- removed L1: 2.2uH, CM5IO:L_Bourns_SRP5030CC
- removed R20: 649R, Resistor_SMD:R_0402_1005Metric
- removed SPI_3: Minifit 2x4, Connector_Molex:Molex_Mini-Fit_Jr_5569-08A2_2x04_P4.20mm_Horizontal
- removed TP5: TestPoint, TestPoint:TestPoint_Pad_2.0x2.0mm
- removed U12: RT9742SNGV, Package_TO_SOT_SMD:TSOT-23_HandSoldering
- removed U18: RT9742GGJ5, Package_TO_SOT_SMD:SOT-23-5
- removed U6: AP22653W6, Package_TO_SOT_SMD:SOT-23-6
- removed U7: ASEK-32.768KHZ-L-R-T, Crystal:Crystal_SMD_3225-4Pin_3.2x2.5mm
- removed U8: TPS54560DDAR, Package_DFN_QFN:DFN-8-1EP_2x2mm_P0.5mm_EP1.05x1.75mm
- J16: footprint CM5IO:Hirose_FH12-22S-0.5SH_1x22-1MP_P0.50mm_Horizontal -> Connector_Molex:Molex_Micro-Fit_3.0_43650-0215_1x02_P3.00mm_Vertical
- J5: footprint CM5IO:Hirose_FH12-22S-0.5SH_1x22-1MP_P0.50mm_Horizontal -> CM5IO:MTCONN_UBAF30-D2011
- J9: footprint Connector_PinHeader_2.54mm:PinHeader_2x02_P2.54mm_Vertical -> Connector_JST:JST_SH_BM04B-SRSS-TB_1x04-1MP_P1.00mm_Vertical
- TP1, TP2, TP3, TP4: moved to F.Cu
- U3: footprint CM5IO:TRJG0926HENL -> Package_SON:USON-10_2.5x1.0mm_P0.5mm
- moved J11 227.1 mm to (21.6, 87.3)
- moved SPI_1 220.3 mm to (30.2, 99.9), turned to 0 degrees
- moved J7 210.8 mm to (69.4, 36.2), turned to 0 degrees
- moved C4 208.8 mm to (24.3, 78.8)
- moved H1 197.2 mm to (82.9, 122.1)
- moved H4 191.6 mm to (89.1, 128.4)
- moved H3 190.8 mm to (89.1, 122.1)
- moved H2 188.8 mm to (82.9, 128.4), turned to 0 degrees
- moved H5 183.9 mm to (95.4, 122.1)
- moved H6 177.7 mm to (95.4, 128.4), turned to 0 degrees
- moved H8 172.7 mm to (101.6, 128.4), turned to 0 degrees
- moved Module1 172.1 mm to (23.4, 71.8), turned to 0 degrees
- moved H7 171.3 mm to (101.6, 122.1), turned to 0 degrees
- moved J4 168.8 mm to (31.5, 78.1)
- moved C9 168.0 mm to (73.8, 107.0), turned to 0 degrees
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Routing:
- net 24V_INPUT: track 0.00 -> 184.7 mm, vias 0 -> 4
- net (no net): track 62.3 -> 231.7 mm, vias 0 -> 13
- net +24V: track 0.00 -> 138.2 mm, vias 0 -> 4
- net /CM5_GPIO ( Ethernet, GPIO, SDCARD)/GPIO2: track 122.2 -> 0.00 mm, vias 1 -> 0
- net /CM5_HighSpeed/USB2_N: track 71.9 -> 194.2 mm, vias 2 -> 3
- net /PCIe-M2/M2_3v3: track 99.8 -> 0.00 mm, vias 2 -> 0
- net /CM5_HighSpeed/DPHY0_D1_N: track 94.6 -> 0.00 mm, vias 2 -> 0
- net /CM5_HighSpeed/DPHY0_C_N: track 92.4 -> 0.00 mm, vias 2 -> 0
- net /CM5_HighSpeed/DPHY0_C_P: track 92.2 -> 0.00 mm, vias 2 -> 0
- net /CM5_HighSpeed/DPHY0_D1_P: track 94.5 -> 177.7 mm, vias 2 -> 3
- net Net-(U5-LEDG_K): track 0.00 -> 69.0 mm
- net /CM5_GPIO ( Ethernet, GPIO, SDCARD)/SD_PWR: track 68.1 -> 0.00 mm
- net +12V: track 43.5 -> 0.00 mm
- net /+5v: track 22.9 -> 0.00 mm
- net Net-(IC1-DD-[3]): track 22.5 -> 0.00 mm, vias 2 -> 0
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Other:
- board outline removed
- board text removed: "CAM/DISP 0"
- board text removed: "CAM/DISP 1"
- board text removed: "Compute Module 5"
- board text removed: "Ethernet"
- board text removed: "FAN"
- board text removed: "Fit for 1.8V GPIO"
- board text removed: "Fit for 3.3V GPIO"
- board text removed: "Fit jumper to disable eMMC Boot"
- board text removed: "Fit jumper to disable writing to EEPROM"
- board text removed: "Fit two jumpers for CAM/DISP 1"
- board text removed: "HDMI0"
- board text removed: "HDMI1"
- board text removed: "J16"
- board text removed: "J3 : nBT_Dis GND"
- board text removed: "J5"
- board text removed: "PMIC_Enable"
- board text removed: "POE"
- board text removed: "PWR_Button"
- board text removed: "Power Button"
- board text removed: "Power In"
- board text removed: "R2"
- board text removed: "Raspberry Pi HAT"
- board text removed: "SYNC_Out"
- board text removed: "USB Device"
- board text removed: "USB3"
- board text removed: "USB_OTG"
- board text removed: "nWireless_Dis"
